File: TDP4_Controller/TDP4_Controller.kicad_pcb (KiCad board)
At the start: 2 copper layers, 0 parts

Commit message: Add files via upload
Other:
- board text added: "Header pins (8.5mm)"
- board text added: "Pins of Display 3.2"
- board text added: "SLIDER (5.8mm)"
- board text added: "moving bit (15.3mm)"
- board text removed: "SLIDER (10.2mm)"
