File: TDP4_Controller/TDP4_Controller.kicad_sch (KiCad schematic)
At the start: 33 parts, among them J1 NRF24, J2 Conn_01x03, J3 MD240128A6W-FPTLW, Q1 BC547, Q3 BC547, SW1 SW_SPDT, SW2 SW_SPDT, SW3 SW_Push, U1 Pico, U2 L7805

Commit message: Add files via upload
Parts:
- removed J2: Conn_01x03, Connector_PinSocket_1.00mm:PinSocket_1x03_P1.00mm_Vertical, symbol Connector_Generic:Conn_01x03
- BT2: footprint (none) -> Connector_PinHeader_2.54mm:PinHeader_1x02_P2.54mm_Vertical
- C1, C2: footprint (none) -> Capacitor_THT:CP_Radial_Tantal_D6.0mm_P2.50mm
- C3, C4, C5: footprint (none) -> Capacitor_THT:C_Disc_D5.0mm_W2.5mm_P5.00mm
- D1, D5: footprint (none) -> Diode_THT:D_A-405_P7.62mm_Horizontal
- D2, D3, D4: footprint (none) -> LED_THT:LED_D5.0mm
- J1: footprint (none) -> TDP4:NRF24
- J3: footprint (none) -> Connector_PinHeader_2.54mm:PinHeader_2x09_P2.54mm_Vertical
- Q3: footprint Package_TO_SOT_THT:TO-92_Inline -> Package_TO_SOT_THT:TO-92
- R1, R10, R11, R2, R3, R4, R5, R6, R7, R8, R9: footprint (none) -> Resistor_THT:R_Axial_DIN0207_L6.3mm_D2.5mm_P10.16mm_Horizontal
- RV1: footprint (none) -> TDP4:Slider.v2
- SW3: footprint (none) -> Button_Switch_THT:SW_PUSH-12mm
- U1: footprint MCU_RaspberryPi_and_Boards:RPi_Pico_SMD_TH -> TDP4:RPi_PicoW_SMD_TH
- U2: footprint (none) -> Package_TO_SOT_THT:TO-220-3_Horizontal_TabDown
Connections:
- net D0: now also U1.1 (GPIO0)
- net D1: now also U1.2 (GPIO1)
- net at R2.2: now also U1.31 (GPIO26_ADC0); no longer U1.20 (GPIO15)
- net at R4.1: now also U1.20 (GPIO15); no longer U1.31 (GPIO26_ADC0)
- no-connect marks 17 -> 20
Other:
- moved on the sheet: C1, C3, D4, J1, R2, R4, R5, R6, RV1, SW3
